Commit message: Added 4 bots with controllers with common launch file

File: src/swarm_simulation/urdf/greybot.xacro (robot description, xacro)
@@ -9,5 +9,5 @@
         <!-- <xacro:box_inertia m = "0.80" x = "0.085" y = "-0.10" z = "0.05" /> -->
         <inertial>
-            <origin rpy="0 0 0" xyz="0.085 -0.10 0.05" />
+            <origin rpy="0 0 0" xyz="0 0 0" />
             <mass value="0.9" />
             <inertia ixx="0.000070003" ixy="0.0" ixz="0.0" iyy="0.000070003" iyz="0.0" izz="0.000040" />
@@ -37,5 +37,5 @@
     name="front"
     color="0 1 0"
-    xyz="0.087 -0.0395 0.0265"
+    xyz="0 0.0585 -.0735"
     rpy="1.570796326794896 0.05 0"/>
     <!-- Rear wheel link -->
@@ -43,5 +43,5 @@
     name="rear"
     color="0 1 0"
-    xyz="0.087 -0.1575 0.0265"
+    xyz="0 -0.0595 -.0735"
     rpy="1.570796326794896 0.05 3.14"/>
     <!-- Left wheel link -->
@@ -49,5 +49,5 @@
     name="left"
     color="0 1 0"
-    xyz="0.0278 -0.099 0.0265"
+    xyz="0.0585 0 -.0735"
     rpy="1.570796326794896 0.05 1.57"/>
     <!-- Right Wheel link  -->
@@ -55,6 +55,6 @@
     name="right"
     color="0 1 0"
-    xyz="0.146 -0.099 0.0265"
-    rpy="1.570796326794896 0.05 -1.57"/>
+    xyz="-0.0590 0 -.0735"
+    rpy="1.570796326794896 0.05 1.57"/>
     <!-- Should install sudo apt-get install ros-noetic-ros-control ros-noetic-ros-controllers -->
     <gazebo>

File: src/swarm_simulation/urdf/redbot.xacro (robot description, xacro)
@@ -9,5 +9,5 @@
         <!-- <xacro:box_inertia m = "0.80" x = "0.085" y = "-0.10" z = "0.05" /> -->
         <inertial>
-            <origin rpy="0 0 0" xyz="0.085 -0.10 0.05" />
+            <origin rpy="0 0 0" xyz="0 0 0" />
             <mass value="0.9" />
             <inertia ixx="0.000070003" ixy="0.0" ixz="0.0" iyy="0.000070003" iyz="0.0" izz="0.000040" />
@@ -37,5 +37,5 @@
     name="front"
     color="0 1 0"
-    xyz="0.087 -0.0395 0.0265"
+    xyz="0 0.0585 -.0735"
     rpy="1.570796326794896 0.05 0"/>
     <!-- Rear wheel link -->
@@ -43,5 +43,5 @@
     name="rear"
     color="0 1 0"
-    xyz="0.087 -0.1575 0.0265"
+    xyz="0 -0.0595 -.0735"
     rpy="1.570796326794896 0.05 3.14"/>
     <!-- Left wheel link -->
@@ -49,16 +49,16 @@
     name="left"
     color="0 1 0"
-    xyz="0.0278 -0.099 0.0265"
-    rpy="1.570796326794896 0.05 1.57"/>
+    xyz="0.0585 0 -.0735"
+    rpy="1.570796326794896 0.05 -1.57"/>
     <!-- Right Wheel link  -->
     <xacro:rim_macro
     name="right"
     color="0 1 0"
-    xyz="0.146 -0.099 0.0265"
-    rpy="1.570796326794896 0.05 -1.57"/>
+    xyz="-0.0590 0 -.0735"
+    rpy="1.570796326794896 0.05 1.57"/>
     <!-- Should install sudo apt-get install ros-noetic-ros-control ros-noetic-ros-controllers -->
     <gazebo>
 		<plugin name="gazebo_ros_control" filename="libgazebo_ros_control.so">
-		<robotNamespace>/redbot</robotNamespace>
+		<robotNamespace>redbot</robotNamespace>
 		</plugin>
 	</gazebo>
